File: BLUEPILL_ENCODER.kicad_sch (KiCad schematic)
At the start: 33 parts, among them J1 boot, J2 Conn_01x04, J3 USB_C_Receptacle_USB2.0_16P, J4 Conn_01x08, SW1 RESET_SWITCH, U1 STM32F103C8T6, U2 AMS1117-3.3, U4 AS5600L-ASOM, Y2 8Mz

Commit message: Add files via upload
Parts:
- C5, C6: footprint Capacitor_Tantalum_SMD:CP_EIA-3528-21_Kemet-B_HandSolder -> Capacitor_SMD:C_0603_1608Metric_Pad1.08x0.95mm_HandSolder
Changed lines of the file:
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@@
 	(text "DECOUPLING & FILTERING\n"
 		(exclude_from_sim no)
-		(at 195.834 22.86 0)
+		(at 243.84 49.784 0)
 		(effects
 			(font
@@
 			)
 		)
-		(property "Footprint" "Capacitor_Tantalum_SMD:CP_EIA-3528-21_Kemet-B_HandSolder"
+		(property "Footprint" "Capacitor_SMD:C_0603_1608Metric_Pad1.08x0.95mm_HandSolder"
 			(at 130.5052 38.1 0)
 			(effects
@@
 			)
 		)
-		(property "Footprint" "Capacitor_Tantalum_SMD:CP_EIA-3528-21_Kemet-B_HandSolder"
+		(property "Footprint" "Capacitor_SMD:C_0603_1608Metric_Pad1.08x0.95mm_HandSolder"
 			(at 106.3752 38.1 0)
 			(effects
@@
 		(on_board yes)
 		(dnp no)
-		(fields_autoplaced yes)
 		(property "Reference" "Y2"
 			(at 99.06 153.67 0)
@@
 					(size 1.27 1.27)
 				)
+				(hide yes)
 			)
 		)
 		(property "Value" "8Mz"
-			(at 99.06 156.21 0)
+			(at 99.06 157.226 0)
 			(effects
 				(font

Commit message: Add files via upload
Pcb is ready, free from critical errors
Ready for manufacturing
Parts:
- removed C12, C13: 1u, Capacitor_SMD:C_0603_1608Metric_Pad1.08x0.95mm_HandSolder, symbol Device:C
- removed C7: 100n, Capacitor_SMD:C_0603_1608Metric_Pad1.08x0.95mm_HandSolder, symbol Device:C
- removed FB1: 120R, FERRITE_BEAD:BEADC2012X105N, symbol Device:FerriteBead
Connections:
- net 3.3v_VDDA_FILTERED is gone; now on net 3.3V_MAIN_POWER_RAIL: U1.9 (VDDA)
Other:
- moved on the sheet: C1, C2, C3, C4

Commit message: Add files via upload
Parts:
- U4: footprint AS5600:SOIC8_AS5600_OSR -> ul_AS5600L-ASOM:AS5600L-ASOM_AMS
Changed lines of the file:
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@@
 			)
 		)
-		(property "Footprint" "AS5600:SOIC8_AS5600_OSR"
+		(property "Footprint" "ul_AS5600L-ASOM:AS5600L-ASOM_AMS"
 			(at 49.53 81.28 0)
 			(effects

Commit message: Add files via upload
SIGNIFICANTLY REDUCED TRACE LENGTH OF I2C PULL-UPs 
AND ERRORS RECTIFIED
Parts:
- R1, R2, R3, R4, R5, R6, R7, R8, R9: footprint Resistor_SMD:R_0805_2012Metric_Pad1.20x1.40mm_HandSolder -> Resistor_SMD:R_0603_1608Metric_Pad0.98x0.95mm_HandSolder
Changed lines of the file:
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@@
 			)
 		)
-		(property "Footprint" "Resistor_SMD:R_0805_2012Metric_Pad1.20x1.40mm_HandSolder"
+		(property "Footprint" "Resistor_SMD:R_0603_1608Metric_Pad0.98x0.95mm_HandSolder"
 			(at 167.64 77.978 90)
 			(effects
@@
 			)
 		)
-		(property "Footprint" "Resistor_SMD:R_0805_2012Metric_Pad1.20x1.40mm_HandSolder"
+		(property "Footprint" "Resistor_SMD:R_0603_1608Metric_Pad0.98x0.95mm_HandSolder"
 			(at 145.542 133.35 90)
 			(effects
@@
 			)
 		)
-		(property "Footprint" "Resistor_SMD:R_0805_2012Metric_Pad1.20x1.40mm_HandSolder"
+		(property "Footprint" "Resistor_SMD:R_0603_1608Metric_Pad0.98x0.95mm_HandSolder"
 			(at 167.132 90.17 90)
 			(effects
@@
 			)
 		)
-		(property "Footprint" "Resistor_SMD:R_0805_2012Metric_Pad1.20x1.40mm_HandSolder"
+		(property "Footprint" "Resistor_SMD:R_0603_1608Metric_Pad0.98x0.95mm_HandSolder"
 			(at 51.562 27.94 90)
 			(effects
@@
 			)
 		)
-		(property "Footprint" "Resistor_SMD:R_0805_2012Metric_Pad1.20x1.40mm_HandSolder"
+		(property "Footprint" "Resistor_SMD:R_0603_1608Metric_Pad0.98x0.95mm_HandSolder"
 			(at 76.962 129.54 90)
 			(effects
@@
 			)
 		)
-		(property "Footprint" "Resistor_SMD:R_0805_2012Metric_Pad1.20x1.40mm_HandSolder"
+		(property "Footprint" "Resistor_SMD:R_0603_1608Metric_Pad0.98x0.95mm_HandSolder"
 			(at 101.092 95.25 90)
 			(effects
@@
 			)
 		)
-		(property "Footprint" "Resistor_SMD:R_0805_2012Metric_Pad1.20x1.40mm_HandSolder"
+		(property "Footprint" "Resistor_SMD:R_0603_1608Metric_Pad0.98x0.95mm_HandSolder"
 			(at 93.472 95.25 90)
 			(effects
@@
 			)
 		)
-		(property "Footprint" "Resistor_SMD:R_0805_2012Metric_Pad1.20x1.40mm_HandSolder"
+		(property "Footprint" "Resistor_SMD:R_0603_1608Metric_Pad0.98x0.95mm_HandSolder"
 			(at 167.64 75.438 90)
 			(effects
@@
 			)
 		)
-		(property "Footprint" "Resistor_SMD:R_0805_2012Metric_Pad1.20x1.40mm_HandSolder"
+		(property "Footprint" "Resistor_SMD:R_0603_1608Metric_Pad0.98x0.95mm_HandSolder"
 			(at 156.972 133.35 90)
 			(effects
